File: pcb/eye-of-terror.kicad_pcb (KiCad board)
At the start: 2 copper layers, 200 x 200 mm, 0 parts

Commit message: WIP layout, most components placed
Parts:
- added C1: 10uF, Capacitor_SMD:CP_Elec_5x5.4, F.Cu at (352.0, 191.2)
- added C10: 100nF, Capacitor_SMD:C_0603_1608Metric, F.Cu at (436.1, 272.4)
- added C11: 100nF, Capacitor_SMD:C_0603_1608Metric, F.Cu at (436.1, 275.0)
- added C12: 15pF, Capacitor_SMD:C_0402_1005Metric, F.Cu at (303.0, 149.5)
- added C13: 15pF, Capacitor_SMD:C_0402_1005Metric, F.Cu at (301.0, 152.5)
- added C14: 100nF, Capacitor_SMD:C_0603_1608Metric, F.Cu at (440.1, 254.9)
- added C15: 100nF, Capacitor_SMD:C_0603_1608Metric, F.Cu at (314.8, 158.8)
- added C16: 4.7uF, Capacitor_SMD:C_0603_1608Metric, F.Cu at (306.6, 152.6)
- added C17: 100nF, Capacitor_SMD:C_0603_1608Metric, F.Cu at (314.9, 142.3)
- added C18: 4.7uF, Capacitor_SMD:C_0603_1608Metric, F.Cu at (321.1, 155.7)
- added C19: 4.7uF, Capacitor_SMD:C_0603_1608Metric, F.Cu at (321.8, 157.9)
- added C2: 100nF, Capacitor_SMD:C_0603_1608Metric, F.Cu at (357.2, 184.0)
- added C20: 4.7uF, Capacitor_SMD:C_0603_1608Metric, F.Cu at (322.6, 155.7)
- added C21: 100nF, Capacitor_SMD:C_0603_1608Metric, F.Cu at (323.6, 150.1)
- added C22: 100nF, Capacitor_SMD:C_0603_1608Metric, F.Cu at (318.7, 158.8)
- added C23: 100nF, Capacitor_SMD:C_0603_1608Metric, F.Cu at (312.7, 142.3)
- added C24: 100nF, Capacitor_SMD:C_0603_1608Metric, F.Cu at (316.8, 142.3)
- added C25: 100nF, Capacitor_SMD:C_0603_1608Metric, F.Cu at (306.6, 148.0)
- added C26: 100nF, Capacitor_SMD:C_0603_1608Metric, F.Cu at (306.6, 149.9)
- added C27: 100nF, Capacitor_SMD:C_0603_1608Metric, F.Cu at (308.7, 157.7)
- added C28: 100nF, Capacitor_SMD:C_0603_1608Metric, F.Cu at (313.3, 158.8)
- added C29: 100nF, Capacitor_SMD:C_0603_1608Metric, F.Cu at (323.6, 148.2)
- added C3: 22uF, Capacitor_SMD:C_0603_1608Metric, F.Cu at (358.1, 190.1)
- added C30: 100nF, Capacitor_SMD:C_0603_1608Metric, F.Cu at (179.9, 168.8)
- added C31: 1uF, Capacitor_SMD:C_0603_1608Metric, F.Cu at (179.9, 171.3)
- added C32: 47nF, Capacitor_SMD:C_0402_1005Metric, F.Cu at (189.0, 168.8)
- added C33: 1uF, Capacitor_SMD:C_0603_1608Metric, F.Cu at (186.2, 163.1)
- added C34: 1uF, Capacitor_SMD:C_0603_1608Metric, F.Cu at (181.2, 164.3)
- added C35: 1uF, Capacitor_SMD:C_0603_1608Metric, F.Cu at (185.0, 167.2)
- added C36: 100nF, Capacitor_SMD:C_0603_1608Metric, F.Cu at (285.9, 90.8)
- added C37: 100nF, Capacitor_SMD:C_0603_1608Metric, F.Cu at (285.9, 93.3)
- added C38: 100nF, Capacitor_SMD:C_0603_1608Metric, F.Cu at (285.9, 95.8)
- added C39: 10uF, Capacitor_SMD:CP_Elec_5x5.4, F.Cu at (292.4, 94.2)
- added C4: 22uF, Capacitor_SMD:C_0603_1608Metric, F.Cu at (352.9, 186.6)
- added C5: 680pF, Capacitor_SMD:C_0402_1005Metric, F.Cu at (351.8, 206.6)
- added C6: 68pF, Capacitor_SMD:C_0603_1608Metric, F.Cu at (351.9, 208.7)
- added C7: 22uF, Capacitor_SMD:C_0603_1608Metric, F.Cu at (354.4, 197.6)
- added C8: 4.7uF, Capacitor_SMD:C_0603_1608Metric, F.Cu at (361.5, 204.2)
- added C9: 100nF, Capacitor_SMD:C_0603_1608Metric, F.Cu at (354.6, 201.6)
- added D1: SM6T30A, Diode_SMD:D_SMB, F.Cu at (392.7, 306.9)
- added D10: RED, Diode_SMD:D_1206_3216Metric, F.Cu at (384.9, 188.6)
- added D11: RED, Diode_SMD:D_1206_3216Metric, F.Cu at (384.9, 192.0)
- added D12: GREEN, Diode_SMD:D_1206_3216Metric, F.Cu at (384.9, 195.4)
- added D13: GREEN, Diode_SMD:D_1206_3216Metric, F.Cu at (384.9, 198.8)
- added D14: GREEN, Diode_SMD:D_1206_3216Metric, F.Cu at (384.9, 202.2)
- added D15: BLUE, Diode_SMD:D_1206_3216Metric, F.Cu at (384.9, 205.4)
- added D16: BLUE, Diode_SMD:D_1206_3216Metric, F.Cu at (384.9, 208.8)
- added D17: BLUE, Diode_SMD:D_1206_3216Metric, F.Cu at (384.9, 212.2)
- added D18: RED, Diode_SMD:D_1206_3216Metric, F.Cu at (368.7, 249.5)
- added D2: SS36, Diode_SMD:D_SMB, F.Cu at (359.1, 200.9)
- added D3: GREEN, Diode_SMD:D_1206_3216Metric, F.Cu at (234.9, 184.1)
- added D4: BLUE, Diode_SMD:D_1206_3216Metric, F.Cu at (235.0, 187.1)
- added D5: GREEN, Diode_SMD:D_1206_3216Metric, F.Cu at (234.9, 192.0)
- added D6: BLUE, Diode_SMD:D_1206_3216Metric, F.Cu at (235.0, 195.0)
- added D7: GREEN, Diode_SMD:D_1206_3216Metric, F.Cu at (235.0, 199.8)
- added D8: BLUE, Diode_SMD:D_1206_3216Metric, F.Cu at (235.1, 202.8)
- added D9: RED, Diode_SMD:D_1206_3216Metric, F.Cu at (384.9, 185.2)
- added H1: MountingHole, MountingHole:MountingHole_3.2mm_M3, F.Cu at (263.1, 117.5)
- added H10: MountingHole, MountingHole:MountingHole_3.2mm_M3, F.Cu at (273.3, 112.6)
- added H11: MountingHole, MountingHole:MountingHole_3.2mm_M3, F.Cu at (216.1, 211.7)
- added H12: MountingHole, MountingHole:MountingHole_3.2mm_M3, F.Cu at (224.0, 238.4)
- added H13: MountingHole, MountingHole:MountingHole_3.2mm_M3, F.Cu at (232.3, 252.8)
- added H14: MountingHole, MountingHole:MountingHole_3.2mm_M3, F.Cu at (239.3, 261.7)
- added H15: MountingHole, MountingHole:MountingHole_3.2mm_M3, F.Cu at (251.5, 272.9)
- added H16: MountingHole, MountingHole:MountingHole_3.2mm_M3, F.Cu at (260.9, 279.3)
- added H17: MountingHole, MountingHole:MountingHole_3.2mm_M3, F.Cu at (275.8, 286.5)
- added H18: MountingHole, MountingHole:MountingHole_3.2mm_M3, F.Cu at (286.6, 289.9)
- added H19: MountingHole, MountingHole:MountingHole_3.2mm_M3, F.Cu at (289.2, 107.7)
- added H2: MountingHole, MountingHole:MountingHole_3.2mm_M3, F.Cu at (249.4, 126.9)
- added H20: MountingHole, MountingHole:MountingHole_3.2mm_M3, F.Cu at (303.0, 292.3)
- added H21: MountingHole, MountingHole:MountingHole_3.2mm_M3, F.Cu at (314.4, 292.3)
- added H22: MountingHole, MountingHole:MountingHole_3.2mm_M3, F.Cu at (330.8, 289.9)
- added H23: MountingHole, MountingHole:MountingHole_3.2mm_M3, F.Cu at (341.6, 286.5)
- added H24: MountingHole, MountingHole:MountingHole_3.2mm_M3, F.Cu at (356.5, 279.3)
- added H25: MountingHole, MountingHole:MountingHole_3.2mm_M3, F.Cu at (365.9, 272.9)
- added H26: MountingHole, MountingHole:MountingHole_3.2mm_M3, F.Cu at (378.1, 261.7)
- added H27: MountingHole, MountingHole:MountingHole_3.2mm_M3, F.Cu at (385.1, 252.8)
- added H28: MountingHole, MountingHole:MountingHole_3.2mm_M3, F.Cu at (300.4, 106.0)
- added H29: MountingHole, MountingHole:MountingHole_3.2mm_M3, F.Cu at (393.4, 238.4)
- added H3: MountingHole, MountingHole:MountingHole_3.2mm_M3, F.Cu at (241.1, 134.6)
- added H30: MountingHole, MountingHole:MountingHole_3.2mm_M3, F.Cu at (397.6, 227.9)
- added H31: MountingHole, MountingHole:MountingHole_3.2mm_M3, F.Cu at (401.3, 211.7)
- added H32: MountingHole, MountingHole:MountingHole_3.2mm_M3, F.Cu at (402.1, 200.4)
- added H33: MountingHole, MountingHole:MountingHole_3.2mm_M3, F.Cu at (400.9, 183.9)
- added H34: MountingHole, MountingHole:MountingHole_3.2mm_M3, F.Cu at (398.4, 172.8)
- added H35: MountingHole, MountingHole:MountingHole_3.2mm_M3, F.Cu at (392.3, 157.4)
- added H36: MountingHole, MountingHole:MountingHole_3.2mm_M3, F.Cu at (386.6, 147.5)
- added H37: MountingHole, MountingHole:MountingHole_3.2mm_M3, F.Cu at (317.0, 106.0)
- added H38: MountingHole, MountingHole:MountingHole_3.2mm_M3, F.Cu at (376.3, 134.6)
- added H39: MountingHole, MountingHole:MountingHole_3.2mm_M3, F.Cu at (368.0, 126.9)
- added H4: MountingHole, MountingHole:MountingHole_3.2mm_M3, F.Cu at (230.8, 147.5)
- added H40: MountingHole, MountingHole:MountingHole_3.2mm_M3, F.Cu at (354.3, 117.5)
- added H41: MountingHole, MountingHole:MountingHole_3.2mm_M3, F.Cu at (344.1, 112.6)
- added H42: MountingHole, MountingHole:MountingHole_3.2mm_M3, F.Cu at (340.2, 144.5)
- added H43: MountingHole, MountingHole:MountingHole_3.2mm_M3, F.Cu at (308.7, 136.1)
- added H44: MountingHole, MountingHole:MountingHole_3.2mm_M3, F.Cu at (277.2, 144.5)
- added H45: MountingHole, MountingHole:MountingHole_3.2mm_M3, F.Cu at (254.1, 167.6)
- added H46: MountingHole, MountingHole:MountingHole_3.2mm_M3, F.Cu at (328.2, 107.7)
- added H47: MountingHole, MountingHole:MountingHole_3.2mm_M3, F.Cu at (245.7, 199.1)
- added H48: MountingHole, MountingHole:MountingHole_3.2mm_M3, F.Cu at (254.1, 230.6)
- added H49: MountingHole, MountingHole:MountingHole_3.2mm_M3, F.Cu at (277.2, 253.6)
- added H5: MountingHole, MountingHole:MountingHole_3.2mm_M3, F.Cu at (225.1, 157.4)
- added H50: MountingHole, MountingHole:MountingHole_3.2mm_M3, F.Cu at (308.7, 262.1)
- added H51: MountingHole, MountingHole:MountingHole_3.2mm_M3, F.Cu at (340.2, 253.6)
- added H52: MountingHole, MountingHole:MountingHole_3.2mm_M3, F.Cu at (363.3, 230.6)
- added H53: MountingHole, MountingHole:MountingHole_3.2mm_M3, F.Cu at (371.7, 199.1)
- added H54: MountingHole, MountingHole:MountingHole_3.2mm_M3, F.Cu at (363.3, 167.6)
- added H6: MountingHole, MountingHole:MountingHole_3.2mm_M3, F.Cu at (219.0, 172.8)
- added H7: MountingHole, MountingHole:MountingHole_3.2mm_M3, F.Cu at (216.5, 183.9)
- added H8: MountingHole, MountingHole:MountingHole_3.2mm_M3, F.Cu at (215.3, 200.4)
- added H9: MountingHole, MountingHole:MountingHole_3.2mm_M3, F.Cu at (219.8, 227.9)
- added J1: Conn_01x02_Socket, Connector_AMASS:AMASS_XT60-M_1x02_P7.20mm_Vertical, F.Cu at (294.6, 250.2)
- added J10: Conn_01x03, Connector_PinHeader_2.54mm:PinHeader_1x03_P2.54mm_Vertical, F.Cu at (387.6, 296.7)
- added J11: Conn_01x03, Connector_PinHeader_2.54mm:PinHeader_1x03_P2.54mm_Vertical, F.Cu at (392.2, 296.7)
- added J12: Conn_01x03, Connector_PinHeader_2.54mm:PinHeader_1x03_P2.54mm_Vertical, F.Cu at (396.8, 296.7)
- added J13: Conn_01x03, Connector_PinHeader_2.54mm:PinHeader_1x03_P2.54mm_Vertical, F.Cu at (401.4, 296.7)
- added J14: Conn_01x03, Connector_PinHeader_2.54mm:PinHeader_1x03_P2.54mm_Vertical, F.Cu at (406.0, 296.7)
- added J15: Conn_01x03, Connector_PinHeader_2.54mm:PinHeader_1x03_P2.54mm_Vertical, F.Cu at (410.6, 296.7)
- added J16: Conn_01x03, Connector_PinHeader_2.54mm:PinHeader_1x03_P2.54mm_Vertical, F.Cu at (415.1, 296.7)
- added J2: G-Switch GT-USB-7055E, ul_GT-USB-7055A:CONN_GT-USB-7055A_GSW, F.Cu at (335.6, 153.2)
- added J3: Conn_01x04, Connector_PinHeader_1.00mm:PinHeader_1x04_P1.00mm_Vertical, B.Cu at (357.1, 141.4)
- added J4: Conn_01x04, Connector_PinHeader_1.00mm:PinHeader_1x04_P1.00mm_Vertical, F.Cu at (357.1, 144.0)
- added J5: Conn_01x03, Connector_PinHeader_2.54mm:PinHeader_1x03_P2.54mm_Vertical, F.Cu at (373.8, 296.7)
- added J6: Conn_01x02_Socket, Connector_AMASS:AMASS_XT60-M_1x02_P7.20mm_Vertical, F.Cu at (353.5, 227.4)
- added J7: Conn_01x02_Socket, Connector_AMASS:AMASS_XT60-M_1x02_P7.20mm_Vertical, F.Cu at (321.5, 250.2)
- added J8: Conn_01x03, Connector_PinHeader_2.54mm:PinHeader_1x03_P2.54mm_Vertical, F.Cu at (378.4, 296.7)
- added J9: Conn_01x03, Connector_PinHeader_2.54mm:PinHeader_1x03_P2.54mm_Vertical, F.Cu at (383.0, 296.7)
- added JP1: SolderJumper_2_Bridged, Jumper:SolderJumper-2_P1.3mm_Bridged_RoundedPad1.0x1.5mm, F.Cu at (436.3, 298.3)
- added JP10: SolderJumper_2_Bridged, Jumper:SolderJumper-2_P1.3mm_Bridged_RoundedPad1.0x1.5mm, B.Cu at (249.2, 147.7)
- added JP11: SolderJumper_2_Bridged, Jumper:SolderJumper-2_P1.3mm_Bridged_RoundedPad1.0x1.5mm, B.Cu at (249.2, 151.2)
- added JP12: SolderJumper_2_Bridged, Jumper:SolderJumper-2_P1.3mm_Bridged_RoundedPad1.0x1.5mm, B.Cu at (249.2, 154.8)
- added JP13: SolderJumper_2_Bridged, Jumper:SolderJumper-2_P1.3mm_Bridged_RoundedPad1.0x1.5mm, B.Cu at (253.6, 144.2)
- added JP14: SolderJumper_2_Bridged, Jumper:SolderJumper-2_P1.3mm_Bridged_RoundedPad1.0x1.5mm, B.Cu at (253.6, 147.7)
- added JP15: SolderJumper_2_Bridged, Jumper:SolderJumper-2_P1.3mm_Bridged_RoundedPad1.0x1.5mm, B.Cu at (253.6, 151.2)
- added JP16: SolderJumper_2_Bridged, Jumper:SolderJumper-2_P1.3mm_Bridged_RoundedPad1.0x1.5mm, F.Cu at (362.9, 249.6)
- added JP17: SolderJumper_3_Open, Jumper:SolderJumper-3_P1.3mm_Open_RoundedPad1.0x1.5mm, F.Cu at (374.4, 305.9)
- added JP18: SolderJumper_3_Open, Jumper:SolderJumper-3_P1.3mm_Open_RoundedPad1.0x1.5mm, F.Cu at (374.4, 309.7)
- added JP19: SolderJumper_3_Open, Jumper:SolderJumper-3_P1.3mm_Open_RoundedPad1.0x1.5mm, F.Cu at (374.4, 313.5)
- added JP2: SolderJumper_2_Bridged, Jumper:SolderJumper-2_P1.3mm_Bridged_RoundedPad1.0x1.5mm, F.Cu at (436.3, 301.9)
- added JP20: SolderJumper_3_Open, Jumper:SolderJumper-3_P1.3mm_Open_RoundedPad1.0x1.5mm, F.Cu at (380.0, 305.9)
- added JP21: SolderJumper_3_Open, Jumper:SolderJumper-3_P1.3mm_Open_RoundedPad1.0x1.5mm, F.Cu at (380.0, 309.7)
- added JP22: SolderJumper_3_Open, Jumper:SolderJumper-3_P1.3mm_Open_RoundedPad1.0x1.5mm, F.Cu at (380.0, 313.5)
- added JP23: SolderJumper_3_Open, Jumper:SolderJumper-3_P1.3mm_Open_RoundedPad1.0x1.5mm, F.Cu at (385.7, 305.9)
- added JP24: SolderJumper_3_Open, Jumper:SolderJumper-3_P1.3mm_Open_RoundedPad1.0x1.5mm, F.Cu at (385.7, 309.7)
- added JP25: SolderJumper_3_Open, Jumper:SolderJumper-3_P1.3mm_Open_RoundedPad1.0x1.5mm, F.Cu at (385.7, 313.5)
- added JP3: SolderJumper_2_Bridged, Jumper:SolderJumper-2_P1.3mm_Bridged_RoundedPad1.0x1.5mm, F.Cu at (436.3, 305.4)
- added JP4: SolderJumper_2_Bridged, Jumper:SolderJumper-2_P1.3mm_Bridged_RoundedPad1.0x1.5mm, F.Cu at (436.3, 309.0)
- added JP5: SolderJumper_2_Bridged, Jumper:SolderJumper-2_P1.3mm_Bridged_RoundedPad1.0x1.5mm, F.Cu at (440.6, 298.3)
- added JP6: SolderJumper_2_Bridged, Jumper:SolderJumper-2_P1.3mm_Bridged_RoundedPad1.0x1.5mm, F.Cu at (440.6, 301.9)
- added JP7: SolderJumper_2_Bridged, Jumper:SolderJumper-2_P1.3mm_Bridged_RoundedPad1.0x1.5mm, F.Cu at (440.6, 305.4)
- added JP8: SolderJumper_2_Bridged, Jumper:SolderJumper-2_P1.3mm_Bridged_RoundedPad1.0x1.5mm, F.Cu at (440.6, 309.0)
- added JP9: SolderJumper_2_Bridged, Jumper:SolderJumper-2_P1.3mm_Bridged_RoundedPad1.0x1.5mm, F.Cu at (445.0, 298.3)
- added L1: 4.7uH, inductor-muRataLQH5BPZ4R7NT0L:IND_LQH5BPZ4R7NT0L, F.Cu at (361.7, 186.4)
- added L2: 10uH, Inductor_SMD:L_Sunlord_MWSA0402S, F.Cu at (351.3, 200.9)
- added L3: 3.3uH, ABRACON-AOTA-B201610S3R3-101-T:ABRACON-AOTA-B201610S3R3-101-T, F.Cu at (324.5, 155.0)
- added NT1: NetTie_3, NetTie:NetTie-3_SMD_Pad2.0mm, B.Cu at (283.9, 147.8)
- added Q1: IPT020N10N3, Package_TO_SOT_SMD:Infineon_PG-HSOF-8-1_ThermalVias, F.Cu at (265.6, 135.7)
- added Q2: IPT020N10N3, Package_TO_SOT_SMD:Infineon_PG-HSOF-8-1_ThermalVias, F.Cu at (277.5, 129.5)
- added Q3: IPT020N10N3, Package_TO_SOT_SMD:Infineon_PG-HSOF-8-1_ThermalVias, F.Cu at (288.3, 125.5)
- added Q4: IPT020N10N3, Package_TO_SOT_SMD:Infineon_PG-HSOF-8-1_ThermalVias, F.Cu at (299.7, 123.2)
- added Q5: IPT020N10N3, Package_TO_SOT_SMD:Infineon_PG-HSOF-8-1_ThermalVias, F.Cu at (310.7, 123.2)
- added Q6: IPT020N10N3, Package_TO_SOT_SMD:Infineon_PG-HSOF-8-1_ThermalVias, F.Cu at (322.4, 125.2)
- added R1: 5.1k, Resistor_SMD:R_0402_1005Metric, F.Cu at (333.8, 149.2)
- added R10: 1k, Resistor_SMD:R_0402_1005Metric, F.Cu at (317.3, 278.2)
- added R11: 1k, Resistor_SMD:R_0402_1005Metric, F.Cu at (315.1, 273.9)
- added R12: 33, Resistor_SMD:R_0402_1005Metric, F.Cu at (323.8, 157.7)
- added R13: 27, Resistor_SMD:R_0402_1005Metric, F.Cu at (321.5, 151.6)
- added R14: 27, Resistor_SMD:R_0402_1005Metric, F.Cu at (321.5, 152.6)
- added R15: 1k, Resistor_SMD:R_0402_1005Metric, F.Cu at (183.0, 160.2)
- added R16: 10k, Resistor_SMD:R_0402_1005Metric, F.Cu at (187.6, 158.9)
- added R17: 1m, Resistor_SMD:R_1206_3216Metric, F.Cu at (278.1, 91.0)
- added R18: 1m, Resistor_SMD:R_1206_3216Metric, F.Cu at (278.1, 94.3)
- added R19: 1m, Resistor_SMD:R_1206_3216Metric, F.Cu at (278.1, 97.7)
- added R2: 5.1k, Resistor_SMD:R_0402_1005Metric, F.Cu at (335.9, 156.1)
- added R20: 68k, Resistor_SMD:R_0603_1608Metric, F.Cu at (452.1, 257.4)
- added R21: 10k, Resistor_SMD:R_0402_1005Metric, F.Cu at (455.9, 307.5)
- added R22: 1k, Resistor_SMD:R_0402_1005Metric, F.Cu at (455.9, 309.5)
- added R23: 1.5k, Resistor_SMD:R_1210_3225Metric, F.Cu at (456.9, 269.4)
- added R24: 10k, Resistor_SMD:R_0402_1005Metric, F.Cu at (458.8, 297.6)
- added R25: 68, Resistor_SMD:R_0402_1005Metric, F.Cu at (238.9, 184.2)
- added R26: 15, Resistor_SMD:R_0603_1608Metric, F.Cu at (239.4, 187.1)
- added R27: 68, Resistor_SMD:R_0402_1005Metric, F.Cu at (238.9, 192.0)
- added R28: 15, Resistor_SMD:R_0603_1608Metric, F.Cu at (239.3, 194.9)
- added R29: 68, Resistor_SMD:R_0402_1005Metric, F.Cu at (238.7, 199.8)
- added R3: 1M, Resistor_SMD:R_0603_1608Metric, F.Cu at (351.3, 205.1)
- added R30: 15, Resistor_SMD:R_0603_1608Metric, F.Cu at (239.1, 202.8)
- added R31: 68, Resistor_SMD:R_0402_1005Metric, F.Cu at (391.1, 186.5)
- added R32: 68, Resistor_SMD:R_0402_1005Metric, F.Cu at (391.1, 188.5)
- added R33: 68, Resistor_SMD:R_0402_1005Metric, F.Cu at (391.1, 190.5)
- added R34: 68, Resistor_SMD:R_0402_1005Metric, F.Cu at (391.3, 196.7)
- added R35: 68, Resistor_SMD:R_0402_1005Metric, F.Cu at (391.3, 198.7)
- added R36: 68, Resistor_SMD:R_0402_1005Metric, F.Cu at (391.3, 200.7)
- added R37: 15, Resistor_SMD:R_0603_1608Metric, F.Cu at (391.0, 206.5)
- added R38: 15, Resistor_SMD:R_0603_1608Metric, F.Cu at (391.0, 209.0)
- added R39: 15, Resistor_SMD:R_0603_1608Metric, F.Cu at (391.0, 211.5)
- added R4: 150k, Resistor_SMD:R_0402_1005Metric, F.Cu at (360.1, 209.4)
- added R40: 1.5k, Resistor_SMD:R_1210_3225Metric, F.Cu at (374.1, 249.5)
- added R5: 43k, Resistor_SMD:R_0603_1608Metric, F.Cu at (350.0, 207.5)
- added R6: 22k, Resistor_SMD:R_0603_1608Metric, F.Cu at (358.1, 210.4)
- added R7: 120k, Resistor_SMD:R_0603_1608Metric, F.Cu at (356.4, 210.4)
- added R8: 1k, Resistor_SMD:R_0402_1005Metric, F.Cu at (302.5, 152.1)
- added R9: 10k, Resistor_SMD:R_0402_1005Metric, F.Cu at (452.9, 305.5)
- added SW1: SW_Push, Button_Switch_SMD:SW_Push_SPST_NO_Alps_SKRK, F.Cu at (309.4, 274.5)
- added SW2: SW_Push, Button_Switch_SMD:SW_Push_SPST_NO_Alps_SKRK, F.Cu at (309.4, 278.9)
- added TP1: TestPoint, TestPoint:TestPoint_Pad_D2.5mm, F.Cu at (271.7, 89.5)
- added TP2: TestPoint, TestPoint:TestPoint_Pad_D2.5mm, F.Cu at (271.7, 94.0)
- added TP3: TestPoint, TestPoint:TestPoint_Pad_D2.5mm, F.Cu at (271.7, 98.6)
- added U1: RP2350B, rpi-lib-kicad-rp235x:QFN-80-1EP_10x10mm_P0.4mm_EP3.4x3.4mm_ThermalVias, F.Cu at (314.6, 150.9)
- added U2: TD1660, Techcode-Semicon-TD1660:TD1660-SOIC-8, F.Cu at (356.3, 206.0)
- added U3: AP63205WU-7, AP6320X-WU:SOIC_05WU-7_DIO, F.Cu at (355.9, 186.7)
- added U4: LSM6DS3, Package_LGA:LGA-14_3x2.5mm_P0.5mm_LayoutBorder3x4y, F.Cu at (267.6, 197.1)
- added U5: W25Q32JVSS, Package_SO:SOIC-8_5.3x5.3mm_P1.27mm, F.Cu at (353.9, 174.6)
- added U6: ~, radiomaster-rp2:RP2, F.Cu at (263.1, 215.3)
- added U7: DRV8353HRTAR, TI_DRV8353HRTAR:RTA0040B, F.Cu at (279.4, 155.1)
- added Y1: ABM8-272-T3, Crystal:Crystal_SMD_3225-4Pin_3.2x2.5mm, F.Cu at (300.1, 149.6)
Routing:
- net /USB_DP: track 0.00 -> 21.8 mm, vias 0 -> 3
- net /USB_DM: track 0.00 -> 19.5 mm
- net DGND: track 0.00 -> 16.9 mm, vias 0 -> 1
- net +3V3: track 0.00 -> 14.0 mm
- net +1V1: track 0.00 -> 10.2 mm, vias 0 -> 2
- net Net-(U1-VREG_LX): track 0.00 -> 7.72 mm, vias 0 -> 2
- net Net-(U1-VREG_AVDD): track 0.00 -> 6.50 mm
- net Net-(J2-CC1): track 0.00 -> 3.66 mm
- net VBUS: track 0.00 -> 3.56 mm
- net Net-(J2-CC2): track 0.00 -> 2.23 mm
- net Net-(U1-USB_DP): track 0.00 -> 1.82 mm
- net Net-(U1-USB_DM): track 0.00 -> 1.57 mm
- added copper zone on F.Cu, net +1V1
- added copper zone on F.Cu, net +3V3
- added copper zone on B.Cu, net DGND
- added copper zone on B.Cu, net PGND
Other:
- outline, holes or cut-outs redrawn

Commit message: WIP layout
Parts:
- removed JP8: SolderJumper_2_Bridged, Jumper:SolderJumper-2_P1.3mm_Bridged_RoundedPad1.0x1.5mm
- removed R24: 10k, Resistor_SMD:R_0402_1005Metric
- added NT2: NetTie_2, NetTie:NetTie-2_SMD_Pad2.0mm, B.Cu at (374.6, 185.8)
- added NT3: NetTie_2, NetTie:NetTie-2_SMD_Pad2.0mm, B.Cu at (374.9, 209.0)
- added NT4: NetTie_2, NetTie:NetTie-2_SMD_Pad2.0mm, B.Cu at (383.5, 215.3)
- added NT5: NetTie_2, NetTie:NetTie-2_SMD_Pad2.0mm, B.Cu at (374.6, 195.8)
- added NT6: NetTie_2, NetTie:NetTie-2_SMD_Pad2.0mm, B.Cu at (381.6, 181.3)
- J4, JP1, JP2, JP3, JP9: moved to B.Cu
- moved JP7 203.6 mm to (263.4, 205.2)
- moved JP6 200.6 mm to (266.6, 202.2)
- moved JP9 198.2 mm to (345.5, 126.9), turned to -90 degrees
- moved JP4 196.9 mm to (267.4, 207.8)
- moved JP5 196.3 mm to (267.9, 205.0)
- moved JP1 195.2 mm to (342.9, 126.9), turned to -90 degrees
- moved JP3 191.3 mm to (345.9, 136.8), turned to 90 degrees
- moved JP2 189.6 mm to (342.9, 136.8), turned to 90 degrees
- moved C10 187.3 mm to (267.6, 190.7)
- moved C11 187.3 mm to (267.6, 193.2)
- moved R9 177.7 mm to (369.1, 148.8), turned to 90 degrees
- moved D9 132.6 mm to (293.6, 281.5), turned to 90 degrees
- moved R31 130.8 mm to (294.9, 275.2), turned to 90 degrees
- moved R32 128.0 mm to (296.9, 275.2), turned to 90 degrees
- moved D10 127.9 mm to (297.0, 281.5), turned to 90 degrees
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Connections:
- R9 pad 2: Net-(JP8-B) -> /GPIO0
- U1 pad 49: /BATT_MON -> unconnected-(U1-GPIO40_ADC0-Pad49)
- U1 pad 52: /5V_MON -> unconnected-(U1-GPIO41_ADC1-Pad52)
- U1 pad 53: +3V3 -> unconnected-(U1-GPIO42_ADC2-Pad53)
- U1 pad 54: /SOC -> /SOA
- U1 pad 56: /SOA -> /SOC
- U1 pad 57: unconnected-(U1-GPIO46_ADC6-Pad57) -> /BATT_MON
- U1 pad 58: unconnected-(U1-GPIO47_ADC7-Pad58) -> /5V_MON
- U5 pad 1: Net-(JP8-B) -> /GPIO0
Routing:
- net +3V3: track 14.0 -> 104.2 mm, vias 0 -> 10
- net /RUN: track 0.00 -> 85.3 mm, vias 0 -> 2
- net /QSPI_SS: track 0.00 -> 83.3 mm, vias 0 -> 2
- net +BATT_RAW: track 0.00 -> 66.9 mm
- net /RP2_RX: track 0.00 -> 64.1 mm, vias 0 -> 2
- net /RP2_TX: track 0.00 -> 62.1 mm
- net /GPIO0: track 0.00 -> 54.1 mm, vias 0 -> 2
- net /QSPI_SD0: track 0.00 -> 53.3 mm, vias 0 -> 2
- net /QSPI_SCLK: track 0.00 -> 51.9 mm, vias 0 -> 2
- net /QSPI_SD3: track 0.00 -> 51.9 mm, vias 0 -> 2
- net /QSPI_SD1: track 0.00 -> 51.0 mm, vias 0 -> 2
- net /QSPI_SD2: track 0.00 -> 51.0 mm, vias 0 -> 2
- net +5V: track 0.00 -> 49.7 mm
- net /SOC: track 0.00 -> 47.1 mm, vias 0 -> 2
- net /SOB: track 0.00 -> 45.5 mm, vias 0 -> 2
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- added copper zone on F.Cu, net +BATT

Commit message: re-routed mosfets for better layout
Parts:
- removed NT1: NetTie_3, NetTie:NetTie-3_SMD_Pad2.0mm
- TP1, TP2, TP3: moved to B.Cu
- moved D7 119.1 mm to (324.6, 121.3)
- moved R29 119.1 mm to (328.3, 121.3)
- moved D8 119.1 mm to (324.7, 124.3)
- moved R30 119.1 mm to (328.7, 124.3)
- moved R15 117.7 mm to (300.7, 159.4), turned to 180 degrees
- moved C34 108.0 mm to (288.2, 150.1), turned to -135 degrees
- moved R16 107.5 mm to (295.1, 160.0)
- moved R21 106.8 mm to (371.5, 242.0)
- moved R22 106.8 mm to (371.5, 244.0)
- moved C33 105.3 mm to (290.6, 149.8), turned to -135 degrees
- moved C35 105.0 mm to (289.7, 159.4), turned to -135 degrees
- moved C30 104.8 mm to (283.0, 150.3), turned to -45 degrees
- moved D6 104.4 mm to (312.8, 125.4)
- moved R28 104.4 mm to (317.1, 125.3)
- moved D5 104.4 mm to (312.7, 122.4)
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Connections:
- net AGND renamed /AGND
- U1 pad 3: /INHA -> /INLC
- U1 pad 4: /INLA -> /INHC
- U1 pad 43: /GPIO34 -> /DRIVER_ENABLE
- U1 pad 44: /GPIO35 -> /DRIVER_FAULTn
- U1 pad 45: /DRIVER_ENABLE -> /GPIO36
- U1 pad 6: /INHB -> /INLB
- U1 pad 7: /INLB -> /INHB
- U1 pad 8: /INHC -> /INLA
- U1 pad 9: /INLC -> /INHA
Routing:
- net PGND: track 30.9 -> 163.8 mm, vias 12 -> 23
- net /SPC: track 0.00 -> 80.5 mm, vias 0 -> 1
- net /INHC: track 5.70 -> 73.7 mm, vias 0 -> 1
- net /INLC: track 5.70 -> 72.8 mm, vias 0 -> 1
- net /INHB: track 5.70 -> 68.6 mm, vias 0 -> 1
- net /INLB: track 5.70 -> 67.3 mm, vias 0 -> 1
- net /MOT_C: track 0.00 -> 59.2 mm
- net /GLC: track 0.00 -> 58.7 mm, vias 0 -> 2
- net /INHA: track 3.28 -> 60.0 mm, vias 0 -> 1
- net /INLA: track 3.68 -> 58.8 mm, vias 0 -> 1
- net /MOT_B: track 0.00 -> 54.3 mm
- net /SDA_TOP_IR_TOF: track 0.00 -> 54.3 mm, vias 0 -> 1
- net /IMU_COPI: track 2.34 -> 55.8 mm, vias 0 -> 1
- net /SCL_TOP_IR_TOF: track 0.00 -> 52.9 mm, vias 0 -> 1
- net /SDA_BOT_IR_TOF: track 0.00 -> 52.5 mm, vias 0 -> 1
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Other:
- board text added: "Phase A"
- board text added: "Phase B"
- board text added: "Phase C"

Commit message: updated smaller footprints for some components
added lock files to gitignore
Other:
- copper layers 2 -> 4
Changed lines of the file:
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@@
 	(layers
 		(0 "F.Cu" signal)
+		(4 "In1.Cu" signal)
+		(6 "In2.Cu" signal)
 		(2 "B.Cu" signal)
 		(9 "F.Adhes" user "F.Adhesive")
@@
 			)
 			(layer "dielectric 1"
-				(type "core")
-				(thickness 1.51)
+				(type "prepreg")
+				(thickness 0.1)
 				(material "FR4")
 				(epsilon_r 4.5)
+				(loss_tangent 0.02)
+			)
+			(layer "In1.Cu"
+				(type "copper")
+				(thickness 0.035)
+			)
+			(layer "dielectric 2"
+				(type "core")
+				(thickness 1.24)
+				(material "FR4")
+				(epsilon_r 4.5)
+				(loss_tangent 0.02)
+			)
+			(layer "In2.Cu"
+				(type "copper")
+				(thickness 0.035)
+			)
+			(layer "dielectric 3"
+				(type "prepreg")
+				(thickness 0.1)
+				(material "FR4")
+				(epsilon_r 4.5)

Commit message: added power and ground planes to middle layers
* removed net ties (for now)
* removed extra gpio pin nets
Parts:
- removed D10, D11, D9: RED, Diode_SMD:D_1206_3216Metric
- removed J10, J11, J12, J13, J14, J15, J16, J8, J9: Conn_01x03, Connector_PinHeader_2.54mm:PinHeader_1x03_P2.54mm_Vertical
- removed JP17, JP18, JP19, JP20, JP21, JP22, JP23, JP24, JP25: SolderJumper_3_Open, Jumper:SolderJumper-3_P1.3mm_Open_RoundedPad1.0x1.5mm
- removed NT2, NT3, NT4, NT5, NT6: NetTie_2, NetTie:NetTie-2_SMD_Pad2.0mm
- removed R31, R32, R33: 68, Resistor_SMD:R_0402_1005Metric
- added D19: RED, Diode_SMD:D_1206_3216Metric, F.Cu at (170.6, 225.4)
- added D20: RED, Diode_SMD:D_1206_3216Metric, F.Cu at (170.6, 228.8)
- added D21: RED, Diode_SMD:D_1206_3216Metric, F.Cu at (170.6, 232.2)
- added D22: RED, Diode_SMD:D_1206_3216Metric, F.Cu at (170.6, 235.6)
- added D23: RED, Diode_SMD:D_1206_3216Metric, F.Cu at (170.6, 239.0)
- added D24: RED, Diode_SMD:D_1206_3216Metric, F.Cu at (170.6, 242.4)
- added D25: RED, Diode_SMD:D_1206_3216Metric, F.Cu at (176.2, 225.4)
- added D26: RED, Diode_SMD:D_1206_3216Metric, F.Cu at (176.2, 228.8)
- added D27: RED, Diode_SMD:D_1206_3216Metric, F.Cu at (176.2, 232.2)
- added D28: RED, Diode_SMD:D_1206_3216Metric, F.Cu at (176.2, 235.6)
- added D29: RED, Diode_SMD:D_1206_3216Metric, F.Cu at (176.2, 239.0)
- added Q10: ALS-PT19-315C/L177/TR8, LED_SMD:LED_0603_1608Metric, F.Cu at (181.1, 232.8)
- added Q11: ALS-PT19-315C/L177/TR8, LED_SMD:LED_0603_1608Metric, F.Cu at (181.1, 235.4)
- added Q12: ALS-PT19-315C/L177/TR8, LED_SMD:LED_0603_1608Metric, F.Cu at (181.1, 238.0)
- added Q13: ALS-PT19-315C/L177/TR8, LED_SMD:LED_0603_1608Metric, F.Cu at (185.1, 225.0)
- added Q14: ALS-PT19-315C/L177/TR8, LED_SMD:LED_0603_1608Metric, F.Cu at (185.1, 227.6)
- added Q15: ALS-PT19-315C/L177/TR8, LED_SMD:LED_0603_1608Metric, F.Cu at (185.1, 230.2)
- added Q16: ALS-PT19-315C/L177/TR8, LED_SMD:LED_0603_1608Metric, F.Cu at (185.1, 232.8)
- added Q17: ALS-PT19-315C/L177/TR8, LED_SMD:LED_0603_1608Metric, F.Cu at (185.1, 235.4)
- added Q7: ALS-PT19-315C/L177/TR8, LED_SMD:LED_0603_1608Metric, F.Cu at (181.1, 225.0)
- added Q8: ALS-PT19-315C/L177/TR8, LED_SMD:LED_0603_1608Metric, F.Cu at (181.1, 227.6)
- added Q9: ALS-PT19-315C/L177/TR8, LED_SMD:LED_0603_1608Metric, F.Cu at (181.1, 230.2)
- added R43: 10k, Resistor_SMD:R_0402_1005Metric, F.Cu at (180.5, 240.2)
- added R44: 68, Resistor_SMD:R_0402_1005Metric, F.Cu at (180.5, 242.2)
- added R45: 68, Resistor_SMD:R_0402_1005Metric, F.Cu at (180.5, 244.2)
- added R46: 10k, Resistor_SMD:R_0402_1005Metric, F.Cu at (180.5, 246.2)
- added R47: 68, Resistor_SMD:R_0402_1005Metric, F.Cu at (180.5, 248.2)
- added R48: 10k, Resistor_SMD:R_0402_1005Metric, F.Cu at (180.5, 250.2)
- added R49: 68, Resistor_SMD:R_0402_1005Metric, F.Cu at (183.4, 240.2)
- added R50: 10k, Resistor_SMD:R_0402_1005Metric, F.Cu at (183.4, 242.2)
- added R51: 68, Resistor_SMD:R_0402_1005Metric, F.Cu at (183.4, 244.2)
- added R52: 68, Resistor_SMD:R_0402_1005Metric, F.Cu at (183.4, 246.2)
- added R53: 68, Resistor_SMD:R_0402_1005Metric, F.Cu at (183.4, 248.2)
- added R54: 68, Resistor_SMD:R_0402_1005Metric, F.Cu at (183.4, 250.2)
- added R55: 10k, Resistor_SMD:R_0402_1005Metric, F.Cu at (186.3, 240.2)
- added R56: 10k, Resistor_SMD:R_0402_1005Metric, F.Cu at (186.3, 242.2)
- added R57: 10k, Resistor_SMD:R_0402_1005Metric, F.Cu at (186.3, 244.2)
- added R58: 10k, Resistor_SMD:R_0402_1005Metric, F.Cu at (186.3, 246.2)
- added R59: 68, Resistor_SMD:R_0402_1005Metric, F.Cu at (186.3, 248.2)
- added R60: 68, Resistor_SMD:R_0402_1005Metric, F.Cu at (186.3, 250.2)
- added R61: 68, Resistor_SMD:R_0402_1005Metric, F.Cu at (189.2, 240.2)
- added R63: 10k, Resistor_SMD:R_0402_1005Metric, F.Cu at (189.2, 242.2)
- added R64: 10k, Resistor_SMD:R_0402_1005Metric, F.Cu at (189.2, 244.2)
- added R65: 10k, Resistor_SMD:R_0402_1005Metric, F.Cu at (189.2, 246.2)
- C10, C11, C14, C15, C16, C17, C18, C19, C20, C21, C22, C23, C24, C25, C26, C27, C28, C29, C8: footprint Capacitor_SMD:C_0603_1608Metric -> Capacitor_SMD:C_0402_1005Metric
- D18: value RED -> GREEN
Connections:
- R21 pad 2: PGND -> DGND
- R23 pad 2: PGND -> DGND
- U1 pad 25: /GPIO24 -> unconnected-(U1-GPIO24-Pad25)
- U1 pad 26: /RED_LED_0 -> unconnected-(U1-GPIO25-Pad26)
- U1 pad 27: /RED_LED_1 -> unconnected-(U1-GPIO26-Pad27)
- U1 pad 28: /RED_LED_2 -> unconnected-(U1-GPIO27-Pad28)
- U1 pad 45: /GPIO36 -> unconnected-(U1-GPIO36-Pad45)
- U1 pad 46: /GPIO37 -> unconnected-(U1-GPIO37-Pad46)
- U1 pad 47: /GPIO38 -> unconnected-(U1-GPIO38-Pad47)
- U1 pad 48: /GPIO39 -> unconnected-(U1-GPIO39-Pad48)
- U1 pad 78: /GPIO1 -> unconnected-(U1-GPIO1-Pad78)
- U1 pad 79: /GPIO2 -> unconnected-(U1-GPIO2-Pad79)
- U1 pad 80: /GPIO3 -> unconnected-(U1-GPIO3-Pad80)
Routing:
- net PGND: track 163.8 -> 52.7 mm
- net +3V3: track 127.2 -> 118.5 mm, vias 14 -> 12
- added copper zone on In1.Cu, net +3V3
- added copper zone on In2.Cu, net DGND
- removed copper zone on F.Cu, net +3V3
- removed copper zone on F.Cu, net +BATT
- removed copper zone on B.Cu, net DGND
- removed copper zone on B.Cu, net PGND
